File: Kicad/MainBot/MainBoard/MainBoard.kicad_pcb (KiCad board)
At the start: 2 copper layers, 116 x 122.5 mm, 99 parts, among them J1 Conn_01x04, J10 Conn_01x04, J11 Conn_01x04, J12 Conn_01x04, J13 01x02_DAC, J14 01x02, J15 Conn_01x24, J16 Conn_01x24, J17 01x24, J18 01x24, J19 01x05, J2 Conn_01x04, J20 01x03, J21 Conn_01x03, J22 Conn_01x03, J23 01x04, J24 01x03, J25 Conn_01x04, J26 01x04, J28 Conn_02x03_Counter_Clockwise, J29 Conn_02x03_Counter_Clockwise, J3 Conn_01x04, J30 Conn_02x03_Counter_Clockwise, J31 Conn_02x03_Counter_Clockwise, J32 Conn_01x03, J33 Conn_01x03, J34 Conn_01x02, J35 Conn_01x02, J36 Conn_01x02, J37 Conn_01x02, J38 Conn_01x03, J39 Conn_01x04, J4 Conn_01x04, J40 Conn_01x03, J41 01x04, J42 01x04, J43 01x04, J44 01x04, J5 02x04_I2C, J6 02x03, J7 02x03, J8 Conn_01x04, J9 Conn_01x04, Q1 Q_PMOS_DGS, U1 TCA9548A, U2 ISL85410, U3 Teensy3.6, U4 DRV8825, U5 DRV8825, U6 DRV8825, U7 DRV8825

Commit message: Small details
Parts:
- moved G*** 2.12 mm to (122.5, 50.5)
Routing:
- net GND: track 121.1 -> 123.5 mm, vias 12 -> 15
- net Net-(C3-Pad1): track 5.79 -> 7.00 mm
Changed lines of the file:
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@@
     (thickness 1.6)
     (drawings 75)
-    (tracks 1266)
+    (tracks 1278)
     (zones 0)
     (modules 99)
@@
   )
   (setup
-    (last_trace_width 0.35)
+    (last_trace_width 0.25)
     (user_trace_width 0.2)
     (user_trace_width 0.25)
@@
   )
   (module Logo:aisler (layer B.Cu)
-    (at 124 49 180)
+    (at 122.5 50.5 180)
     (fp_text reference G*** (at 0 0 180) (layer B.SilkS) hide
       (effects (font (thickness 0.3)) (justify mirror))
@@
     (effects (font (size 1 1) (thickness 0.2)))
   )
+  (via (at 63.3 129) (size 0.6) (drill 0.4) (layers F.Cu B.Cu) (net 1))
+  (segment (start 63.3 129) (end 63.3235 128.9765) (width 0.25) (layer F.Cu) (net 1))
+  (segment (start 63.3235 128.9765) (end 63.3235 127.8705) (width 0.25) (layer F.Cu) (net 1))
+  (via (at 63.3 126.8) (size 0.6) (drill 0.4) (layers F.Cu B.Cu) (net 1))
+  (segment (start 63.3 126.8) (end 63.3235 126.8235) (width 0.25) (layer F.Cu) (net 1))
+  (segment (start 63.3235 126.8235) (end 63.3235 127.8705) (width 0.25) (layer F.Cu) (net 1))
+  (via (at 63.3235 127.8705) (size 0.6) (drill 0.4) (layers F.Cu B.Cu) (net 1))
+  (segment (start 63.3 127.8) (end 63.3 127.894) (width 0.25) (layer B.Cu) (net 1))
+  (segment (start 63.3 127.894) (end 63.3235 127.8705) (width 0.25) (layer B.Cu) (net 1))
   (segment (start 65.5 126) (end 65.8 125.7) (width 0.35) (layer F.Cu) (net 1))
   (via (at 65.8 125.7) (size 0.6) (drill 0.4) (layers F.Cu B.Cu) (net 1))
@@
   (segment (start 67.9735 127.6205) (end 68.0385 127.5555) (width 0.3) (layer F.Cu) (net 41))
   (segment (start 55.87 59.01) (end 55.87 59.3275) (width 0.75) (layer B.Cu) (net 41))
-  (segment (start 64.8221 128.1205) (end 66.05 128.1205) (width 0.3) (layer F.Cu) (net 42))
-  (segment (start 66.816 126.7275) (end 68.4035 125.14) (width 0.3) (layer F.Cu) (net 42))
-  (via (at 66.816 126.7275) (size 0.6) (drill 0.4) (layers F.Cu B.Cu) (net 42))
-  (segment (start 66.816 127.6165) (end 66.816 126.7275) (width 0.3) (layer B.Cu) (net 42))
-  (segment (start 66.181 128.2515) (end 66.816 127.6165) (width 0.3) (layer B.Cu) (net 42))
-  (via (at 66.181 128.2515) (size 0.6) (drill 0.4) (layers F.Cu B.Cu) (net 42))
-  (segment (start 66.05 128.1205) (end 66.181 128.2515) (width 0.3) (layer F.Cu) (net 42))
+  (segment (start 64.8221 128.1205) (end 66.3205 128.1205) (width 0.25) (layer F.Cu) (net 42))
+  (segment (start 67.1 126.5) (end 68.4035 125.1965) (width 0.25) (layer F.Cu) (net 42))
+  (via (at 67.1 126.5) (size 0.6) (drill 0.4) (layers F.Cu B.Cu) (net 42))
+  (segment (start 66.9 126.7) (end 67.1 126.5) (width 0.25) (layer B.Cu) (net 42))
+  (segment (start 66.9 128.5) (end 66.9 126.7) (width 0.25) (layer B.Cu) (net 42))
+  (segment (start 66.8 128.6) (end 66.9 128.5) (width 0.25) (layer B.Cu) (net 42))
+  (via (at 66.8 128.6) (size 0.6) (drill 0.4) (layers F.Cu B.Cu) (net 42))
+  (segment (start 66.3205 128.1205) (end 66.8 128.6) (width 0.25) (layer F.Cu) (net 42))
+  (segment (start 68.4035 125.1965) (end 68.4035 124.7905) (width 0.25) (layer F.Cu) (net 42))
   (segment (start 68.4035 125.14) (end 68.4035 124.7905) (width 0.3) (layer F.Cu) (net 42))
+  (segment (start 61.8249 129.1205) (end 61.8249 130.2249) (width 0.25) (layer F.Cu) (net 43))
+  (segment (start 61.8249 130.2249) (end 62 130.4) (width 0.25) (layer F.Cu) (net 43))
+  (segment (start 61.8249 127.6205) (end 59.9795 127.6205) (width 0.25) (layer F.Cu) (net 43))
+  (segment (start 59.9795 127.6205) (end 59.9 127.7) (width 0.25) (layer F.Cu) (net 43))
+  (via (at 59.9 127.7) (size 0.6) (drill 0.4) (layers F.Cu B.Cu) (net 43))
+  (segment (start 59.9 127.7) (end 59.9 130.2) (width 0.25) (layer B.Cu) (net 43))
+  (via (at 59.9 130.2) (size 0.6) (drill 0.4) (layers F.Cu B.Cu) (net 43))
+  (segment (start 59.9 130.2) (end 60.1 130.4) (width 0.25) (layer F.Cu) (net 43))
+  (segment (start 60.1 130.4) (end 62 130.4) (width 0.25) (layer F.Cu) (net 43))
+  (segment (start 62 130.4) (end 63.26 131.66) (width 0.25) (layer F.Cu) (net 43))
+  (segment (start 63.26 131.66) (end 63.26 132.284) (width 0.25) (layer F.Cu) (net 43))
   (segment (start 63.26 132.284) (end 63.165 132.284) (width 0.3) (layer F.Cu) (net 43))
-  (segment (start 63.165 132.284) (end 60.8724 129.9914) (width 0.3) (layer F.Cu) (net 43))
   (segment (start 64.8221 129.1205) (end 64.8221 130.7219) (width 0.3) (layer F.Cu) (net 43))
   (segment (start 64.8221 130.7219) (end 63.26 132.284) (width 0.3) (layer F.Cu) (net 43))
-  (segment (start 61.8249 127.6205) (end 60.208 127.6205) (width 0.3) (layer F.Cu) (net 43))
-  (segment (start 60.1739 129.9914) (end 60.8724 129.9914) (width 0.3) (layer F.Cu) (net 43))
-  (segment (start 60.8724 129.9914) (end 61.8249 129.9914) (width 0.3) (layer F.Cu) (net 43))
-  (segment (start 59.8945 129.712) (end 60.1739 129.9914) (width 0.3) (layer F.Cu) (net 43))
-  (via (at 59.8945 129.712) (size 0.6) (drill 0.4) (layers F.Cu B.Cu) (net 43))
-  (segment (start 59.8945 127.934) (end 59.8945 129.712) (width 0.3) (layer B.Cu) (net 43))
-  (via (at 59.8945 127.934) (size 0.6) (drill 0.4) (layers F.Cu B.Cu) (net 43))
-  (segment (start 60.208 127.6205) (end 59.8945 127.934) (width 0.3) (layer F.Cu) (net 43))
   (segment (start 61.8249 128.6205) (end 61.8249 129.1205) (width 0.3) (layer F.Cu) (net 43))
-  (segment (start 61.8249 129.1205) (end 61.8249 129.9914) (width 0.3) (layer F.Cu) (net 43))
   (segment (start 63.26 131.4265) (end 63.26 132.284) (width 0.3) (layer F.Cu) (net 43))
   (segment (start 61.8249 128.1205) (end 60.6285 128.1205) (width 0.3) (layer F.Cu) (net 44))
